File: Quantum Board.kicad_pcb (KiCad board)
At the start: 2 copper layers, 130 parts, among them J1 OLED_128x32, U1 Raspberry_Pi_Pico

Commit message: Quantum Board Part 4
Parts:
- D1, D10, D11, D12, D13, D14, D15, D16, D17, D18, D19, D2, D20, D21, D22, D23, D24, D25, D26, D27, D28, D29, D3, D30, D31, D32, D33, D34, D35, D36, D37, D38, D39, D4, D40, D41, D42, D43, D44, D45, D46, D47, D48, D49, D5, D50, D51, D52, D53, D54, D55, D56, D57, D58, D59, D6, D63, D67, D68, D69, D7, D70, D8, D9: moved to B.Cu
- moved D14 531.5 mm to (314.9, 54.2), turned to 90 degrees
- moved D13 525.1 mm to (285.9, 54.2), turned to 90 degrees
- moved D12 505.0 mm to (265.9, 54.2), turned to 90 degrees
- moved S14 498.6 mm to (301.4, 50.4)
- moved D11 484.9 mm to (245.9, 54.2), turned to 90 degrees
- moved S13 471.9 mm to (276.9, 50.4)
- moved D10 464.8 mm to (225.9, 54.2), turned to 90 degrees
- moved S12 450.2 mm to (256.9, 50.4)
- moved D9 444.8 mm to (205.9, 54.2), turned to 90 degrees
- moved S27 434.9 mm to (276.9, 69.3)
- moved S11 428.8 mm to (236.9, 50.4)
- moved D8 424.7 mm to (185.9, 54.2), turned to 90 degrees
- moved S26 414.9 mm to (256.9, 69.3)
- moved S10 408.1 mm to (216.9, 50.4)
- moved S40 404.9 mm to (256.9, 88.3)
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
Commit message: Quantum Board Part 5
Parts:
- added J2: OLED_128x32, ScottoKeebs_Components:OLED_128x32, F.Cu at (141.7, 72.0)
- added J3: OLED_128x32, ScottoKeebs_Components:OLED_128x32, F.Cu at (227.7, 72.0)
- moved D70 283.4 mm to (326.3, 179.2)
- moved D56 274.7 mm to (347.3, 160.2)
- moved D28 272.0 mm to (347.3, 122.2)
- moved D42 271.7 mm to (347.3, 141.2)
- moved D26 264.5 mm to (298.3, 122.2)
- moved D69 259.9 mm to (306.3, 179.2)
- moved D55 242.1 mm to (318.3, 160.2)
- moved D25 241.6 mm to (278.3, 122.2)
- moved D27 240.1 mm to (318.3, 122.2)
- moved D39 239.4 mm to (278.3, 141.2)
- moved D41 239.2 mm to (318.3, 141.2)
- moved D68 236.6 mm to (286.3, 179.2)
- moved D24 218.9 mm to (258.3, 122.2)
- moved D54 218.6 mm to (298.3, 160.2)
- moved D52 217.5 mm to (258.3, 160.2)
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Routing:
- net C14: track 0.00 -> 341.5 mm
- net C12: track 0.00 -> 316.3 mm
- net C11: track 0.00 -> 297.8 mm
- net C10: track 0.00 -> 282.3 mm
- net C9: track 0.00 -> 241.5 mm
- net C8: track 0.00 -> 224.2 mm
- net C6: track 0.00 -> 209.7 mm
- net C7: track 0.00 -> 206.6 mm
- net +5V: track 0.00 -> 203.1 mm
- net C5: track 0.00 -> 174.2 mm
- net C4: track 0.00 -> 159.1 mm
- net GND: track 0.00 -> 158.0 mm
- net C2: track 0.00 -> 146.5 mm
- net C3: track 0.00 -> 139.3 mm
- net SCL: track 0.00 -> 128.5 mm
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Other:
- board outline added: 299.6 x 123.5 mm

Commit message: Quantum Board Part 6
Parts:
- added D60: Diode, ScottoKeebs_Components:Diode_DO-35, F.Cu at (357.0, 207.0)
- added D60: Diode, ScottoKeebs_Components:Diode_DO-35, F.Cu at (452.0, 162.1)
- added D61: Diode, ScottoKeebs_Components:Diode_DO-35, F.Cu at (452.0, 165.6)
- added D62: Diode, ScottoKeebs_Components:Diode_DO-35, F.Cu at (452.0, 169.2)
- added D64: Diode, ScottoKeebs_Components:Diode_DO-35, F.Cu at (452.0, 172.7)
- added D65: Diode, ScottoKeebs_Components:Diode_DO-35, F.Cu at (452.0, 176.2)
- added S61: Keyswitch, ScottoKeebs_Choc:Choc_V1_1.00u, F.Cu at (442.1, 168.6)
- added S62: Keyswitch, ScottoKeebs_Choc:Choc_V1_1.50u, F.Cu at (442.1, 185.1)
- added S63: Keyswitch, ScottoKeebs_Choc:Choc_V1_1.00u, F.Cu at (442.1, 201.7)
- added S64: Keyswitch, ScottoKeebs_Choc:Choc_V1_1.00u, F.Cu at (442.1, 218.2)
- added S65: Keyswitch, ScottoKeebs_Choc:Choc_V1_1.00u, F.Cu at (442.1, 234.8)
- added S65: Keyswitch, ScottoKeebs_Choc:Choc_V1_1.50u, F.Cu at (363.7, 196.9)
- moved D1 7.62 mm to (78.3, 103.2), turned to 90 degrees
Routing:
- net R4: track 0.00 -> 441.5 mm
- net R3: track 0.00 -> 436.8 mm
- net R2: track 0.00 -> 413.8 mm
- net R1: track 0.00 -> 390.7 mm
- net R0: track 0.00 -> 365.8 mm
- net GND: track 158.0 -> 206.3 mm
- net Net-(D63-A): track 0.00 -> 44.5 mm
- net SDA: track 127.8 -> 170.8 mm
- net SCL: track 128.5 -> 171.5 mm
- net Net-(D59-A): track 0.00 -> 8.50 mm
- net Net-(D67-A): track 0.00 -> 8.50 mm
- net Net-(D56-A): track 0.00 -> 8.50 mm
- net Net-(D42-A): track 0.00 -> 8.50 mm
- net Net-(D29-A): track 0.00 -> 8.50 mm
- net Net-(D58-A): track 0.00 -> 8.50 mm
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Other:
- board text added: "Quantum Board"
- board text added: "rev. 1"
